File: mini1284.brd (EAGLE design)
At the start: 64.8 x 20.8 mm, 25 parts, among them U1 ATMEGA644A, Y1 16MHz

Commit message: Further tweaks.
Parts:
- U1: value ATMEGA644A -> ATmega1284P-AU
Changed lines of the file:
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@@
 </autorouter>
 <elements>
-<element name="U1" library="atmel" package="TQFP44" value="ATMEGA644A" x="30.48" y="10.1346" smashed="yes">
+<element name="U1" library="atmel" package="TQFP44" value="ATmega1284P-AU" x="30.48" y="10.1346" smashed="yes">
 <attribute name="OC_NEWARK" value="58M3748" x="57.149990625" y="-0.0254" size="1.778" layer="27" display="off"/>
 <attribute name="MPN" value="ATMEGA644PV-10AU" x="57.149990625" y="-0.0254" size="1.778" layer="27" display="off"/>
