File: mini1284.brd (EAGLE design)
At the start: 64.8 x 20.8 mm, 25 parts, among them U1 ATmega1284P-AU, Y1 16MHz

Commit message: Update ReadMe file, add LICENSE file and photo.
Parts:
- C7, C8: value 27pF -> 22pF
Changed lines of the file:
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@@
 <attribute name="VALUE" x="37.9368" y="9.12" size="0.8128" layer="27" ratio="16" rot="R270"/>
 </element>
-<element name="C7" library="_jc" package="M0805" value="27pF" x="15.24" y="13.716" smashed="yes" rot="R180">
+<element name="C7" library="_jc" package="M0805" value="22pF" x="15.24" y="13.716" smashed="yes" rot="R180">
 <attribute name="NAME" x="11.581" y="13.3872" size="0.8128" layer="25" ratio="16"/>
 <attribute name="VALUE" x="16.74" y="16.216" size="0.8128" layer="27" ratio="16" rot="R180"/>
 </element>
-<element name="C8" library="_jc" package="M0805" value="27pF" x="15.24" y="6.858" smashed="yes" rot="R180">
+<element name="C8" library="_jc" package="M0805" value="22pF" x="15.24" y="6.858" smashed="yes" rot="R180">
 <attribute name="NAME" x="11.5556" y="7.215" size="0.8128" layer="25" ratio="16"/>
 <attribute name="VALUE" x="16.74" y="9.358" size="0.8128" layer="27" ratio="16" rot="R180"/>
