File: mini1284.sch (EAGLE design)
At the start: 37 parts, among them U1 ATMEGA644A

Commit message: Routing looking pretty good.
Parts:
- removed C10, C11, C12: (no value), _jc:C-USM0805
- removed C13: 100nF, _jc:C-USM0805
- removed D2: (no value), _jc:LEDCHIPLED_1206
- removed D3: 1N4148, _jc:DIODESOD-323F
- removed R10, R2, R3, R4, R5, R6, R7, R8, R9: (no value), _jc:R-US_M0805
- removed R11: 10K, _jc:R-US_M0805
- added LOGO2: OSHW_LOGO_6MILX0100-NT, ohw-logo:OSHW_LOGO_6MILX0100-NT
- C1, C2, C3, C4, C5, C9: value (none) -> 100nF
- C6: value (none) -> 10uF; device _jc:C-USM0805 -> _jc:C-USM1206
- C7, C8: value (none) -> 27pF
- D1: value (none) -> 1N4148; device _jc:DIODESOD-323F -> _jc:DIODESOD-323F-A
- L1: value (none) -> 10uH
- R1: value (none) -> 10K
- S1: device _jc:10-XXOCT -> _jc:10-XXPTS810
- Y1: value (none) -> 16MHz
Connections:
- net /RESET: now also C9.1, D1.A, R1.1; no longer C13.1, D3.A, R11.1
- net AREF: now also C5.1; no longer C8.1
- net N$2: now also C8.1; no longer C6.1
- net N$3: now also C7.1; no longer C5.1
- net RST: now also C9.2; no longer C13.2
- net VCC: now also C6.1, D1.K, R1.2; no longer C7.1, D3.K, R11.2
Other:
- note added: "CC BY-SA 4.0"
- note added: "Mighty Mini 1284P"
- note added: "Mighty Mini 1284P by Jack Christensen is licensed under"
- note added: "a Creative Commons Attribution-ShareAlike 4.0 International License."
- note added: "by Jack Christensen"
- note added: "v0.8"
- moved on the sheet: C1, C2, C3, C4, C5, C6, C7, C8, C9, D1, JP1, JP2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

Commit message: Routing refinements.
Parts:
- added D2: LED, _jc:LEDD0805A
- added LOGO1: OSHW_LOGO_8MILX0150-NT, ohw-logo:OSHW_LOGO_8MILX0150-NT
- added R2: 1K, _jc:R-US_M0805
Connections:
- new net N$34: D2.C, R2.2
- net GND: now also R2.1
- net SCK: now also D2.A
Changed lines of the file:
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@@
 <part name="GND4" library="SparkFun" deviceset="GND" device=""/>
 <part name="LOGO2" library="ohw-logo" deviceset="OSHW_LOGO_6MIL" device="X0100-NT" value="OSHW_LOGO_6MILX0100-NT"/>
+<part name="LOGO1" library="ohw-logo" deviceset="OSHW_LOGO_8MIL" device="X0150-NT" value="OSHW_LOGO_8MILX0150-NT"/>
+<part name="R2" library="_jc" deviceset="R-US_" device="M0805" value="1K"/>
+<part name="D2" library="_jc" deviceset="LED" device="D0805A" value="LED"/>
+<part name="GND7" library="SparkFun" deviceset="GND" device=""/>
 </parts>
 <sheets>
@@
 </instance>
 <instance part="LOGO2" gate="G$1" x="10.16" y="17.78"/>
+<instance part="LOGO1" gate="G$1" x="10.16" y="25.4"/>
+<instance part="R2" gate="G$1" x="86.36" y="149.86" smashed="yes" rot="R90">
+<attribute name="NAME" x="87.6554" y="153.924" size="1.778" layer="95"/>
+<attribute name="VALUE" x="87.63" y="151.384" size="1.778" layer="96"/>
+</instance>
+<instance part="D2" gate="G$1" x="86.36" y="162.56"/>
+<instance part="GND7" gate="1" x="86.36" y="139.7" smashed="yes">
+<attribute name="VALUE" x="83.82" y="137.16" size="1.778" layer="96"/>
+</instance>
 </instances>
 <busses>
@@
 <pinref part="GND4" gate="1" pin="GND"/>
 <wire x1="68.58" y1="109.22" x2="68.58" y2="104.14" width="0.1524" layer="91"/>
+</segment>
+<segment>
+<pinref part="R2" gate="G$1" pin="1"/>
+<wire x1="86.36" y1="144.78" x2="86.36" y2="142.24" width="0.1524" layer="91"/>
+<pinref part="GND7" gate="1" pin="GND"/>
 </segment>
 </net>
@@
 <label x="198.12" y="142.24" size="1.778" layer="95"/>
 </segment>
+<segment>
+<pinref part="D2" gate="G$1" pin="A"/>
+<wire x1="86.36" y1="165.1" x2="86.36" y2="167.64" width="0.1524" layer="91"/>
+<wire x1="86.36" y1="167.64" x2="78.74" y2="167.64" width="0.1524" layer="91"/>
+<label x="78.74" y="167.64" size="1.778" layer="95"/>
+</segment>
 </net>
 <net name="MISO" class="0">
@@
 </segment>
 </net>
+<net name="N$34" class="0">
+<segment>
+<pinref part="D2" gate="G$1" pin="C"/>
+<pinref part="R2" gate="G$1" pin="2"/>
+<wire x1="86.36" y1="157.48" x2="86.36" y2="154.94" width="0.1524" layer="91"/>
+</segment>
+</net>

Commit message: Further tweaks.
Parts:
- U1: value ATMEGA644A -> ATmega1284P-AU
Changed lines of the file:
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@@
 <grid distance="0.1" unitdist="inch" unit="inch" style="lines" multiple="1" display="no" altdistance="0.01" altunitdist="inch" altunit="inch"/>
 <layers>
-<layer number="1" name="Top" color="4" fill="1" visible="yes" active="no"/>
-<layer number="16" name="Bottom" color="1" fill="1" visible="yes" active="no"/>
-<layer number="17" name="Pads" color="2" fill="1" visible="yes" active="no"/>
-<layer number="18" name="Vias" color="2" fill="1" visible="yes" active="no"/>
-<layer number="19" name="Unrouted" color="6" fill="1" visible="yes" active="no"/>
-<layer number="20" name="Dimension" color="15" fill="1" visible="yes" active="no"/>
-<layer number="21" name="tPlace" color="7" fill="1" visible="yes" active="no"/>
-<layer number="22" name="bPlace" color="7" fill="1" visible="yes" active="no"/>
-<layer number="23" name="tOrigins" color="15" fill="1" visible="yes" active="no"/>
-<layer number="24" name="bOrigins" color="15" fill="1" visible="yes" active="no"/>
-<layer number="25" name="tNames" color="7" fill="1" visible="yes" active="no"/>
-<layer number="26" name="bNames" color="7" fill="1" visible="yes" active="no"/>
-<layer number="27" name="tValues" color="7" fill="1" visible="yes" active="no"/>
-<layer number="28" name="bValues" color="7" fill="1" visible="yes" active="no"/>
+<layer number="1" name="Top" color="4" fill="1" visible="no" active="no"/>
+<layer number="16" name="Bottom" color="1" fill="1" visible="no" active="no"/>
+<layer number="17" name="Pads" color="2" fill="1" visible="no" active="no"/>
+<layer number="18" name="Vias" color="2" fill="1" visible="no" active="no"/>
+<layer number="19" name="Unrouted" color="6" fill="1" visible="no" active="no"/>
+<layer number="20" name="Dimension" color="15" fill="1" visible="no" active="no"/>
+<layer number="21" name="tPlace" color="7" fill="1" visible="no" active="no"/>
+<layer number="22" name="bPlace" color="7" fill="1" visible="no" active="no"/>
+<layer number="23" name="tOrigins" color="15" fill="1" visible="no" active="no"/>
+<layer number="24" name="bOrigins" color="15" fill="1" visible="no" active="no"/>
+<layer number="25" name="tNames" color="7" fill="1" visible="no" active="no"/>
+<layer number="26" name="bNames" color="7" fill="1" visible="no" active="no"/>
+<layer number="27" name="tValues" color="7" fill="1" visible="no" active="no"/>
+<layer number="28" name="bValues" color="7" fill="1" visible="no" active="no"/>
 <layer number="29" name="tStop" color="7" fill="3" visible="no" active="no"/>
 <layer number="30" name="bStop" color="7" fill="6" visible="no" active="no"/>
@@
 <layer number="35" name="tGlue" color="7" fill="4" visible="no" active="no"/>
 <layer number="36" name="bGlue" color="7" fill="5" visible="no" active="no"/>
-<layer number="37" name="tTest" color="7" fill="1" visible="yes" active="no"/>
-<layer number="38" name="bTest" color="7" fill="1" visible="yes" active="no"/>
+<layer number="37" name="tTest" color="7" fill="1" visible="no" active="no"/>
+<layer number="38" name="bTest" color="7" fill="1" visible="no" active="no"/>
 <layer number="39" name="tKeepout" color="4" fill="11" visible="no" active="no"/>
 <layer number="40" name="bKeepout" color="1" fill="11" visible="no" active="no"/>
@@
 <layer number="44" name="Drills" color="7" fill="1" visible="no" active="no"/>
 <layer number="45" name="Holes" color="7" fill="1" visible="no" active="no"/>
-<layer number="46" name="Milling" color="3" fill="1" visible="yes" active="no"/>
-<layer number="47" name="Measures" color="7" fill="1" visible="yes" active="no"/>
-<layer number="48" name="Document" color="7" fill="1" visible="yes" active="no"/>
-<layer number="49" name="Reference" color="7" fill="1" visible="yes" active="no"/>
-<layer number="50" name="dxf" color="7" fill="1" visible="yes" active="no"/>
-<layer number="51" name="tDocu" color="7" fill="1" visible="yes" active="no"/>
-<layer number="52" name="bDocu" color="7" fill="1" visible="yes" active="no"/>
-<layer number="53" name="tGND_GNDA" color="7" fill="9" visible="yes" active="no"/>
-<layer number="54" name="bGND_GNDA" color="1" fill="9" visible="yes" active="no"/>
-<layer number="56" name="wert" color="7" fill="1" visible="yes" active="no"/>
+<layer number="46" name="Milling" color="3" fill="1" visible="no" active="no"/>
+<layer number="47" name="Measures" color="7" fill="1" visible="no" active="no"/>
+<layer number="48" name="Document" color="7" fill="1" visible="no" active="no"/>
+<layer number="49" name="Reference" color="7" fill="1" visible="no" active="no"/>
+<layer number="50" name="dxf" color="7" fill="1" visible="no" active="no"/>
+<layer number="51" name="tDocu" color="7" fill="1" visible="no" active="no"/>
+<layer number="52" name="bDocu" color="7" fill="1" visible="no" active="no"/>
+<layer number="53" name="tGND_GNDA" color="7" fill="9" visible="no" active="no"/>
+<layer number="54" name="bGND_GNDA" color="1" fill="9" visible="no" active="no"/>
+<layer number="56" name="wert" color="7" fill="1" visible="no" active="no"/>
 <layer number="91" name="Nets" color="2" fill="1" visible="yes" active="yes"/>
 <layer number="92" name="Busses" color="1" fill="1" visible="yes" active="yes"/>
@@
 </classes>
 <parts>
-<part name="U1" library="atmel" deviceset="ATMEGA644" device="A"/>
+<part name="U1" library="atmel" deviceset="ATMEGA644" device="A" value="ATmega1284P-AU"/>
 <part name="C1" library="_jc" deviceset="C-US" device="M0805" value="100nF"/>
 <part name="C2" library="_jc" deviceset="C-US" device="M0805" value="100nF"/>
@@
 <instances>
 <instance part="U1" gate="G$1" x="170.18" y="121.92" smashed="yes">
-<attribute name="VALUE" x="147.32" y="73.66" size="1.778" layer="96"/>
+<attribute name="VALUE" x="167.64" y="168.91" size="1.778" layer="96"/>
 <attribute name="NAME" x="147.32" y="168.91" size="1.778" layer="95"/>
 </instance>
